File: hardware/pcb/TMPM4KNF10AFG.kicad_pcb (KiCad board)
At the start: 4 copper layers, 103.4 x 101 mm, 91 parts, among them J1 Conn_01x02_Socket, J2 Conn_01x02_Socket, J3 Conn_01x02_Socket, J4 Conn_01x06_Pin, J5 Conn_01x03_Pin, J6 Conn_01x06_Pin, J7 Conn_01x06_Pin, J8 Conn_01x04_Pin, Q2 NMOS, Q3 NMOS, Q4 NMOS, Q5 NMOS, SW1 CSS-1210MC, SW2 EVQ-PBG05R, U1 TMPM4KNF10AFG, U2 BD9C301FJ-E2, U4 TB67H450AFNG_EL, U5 TB67H450AFNG_EL

Commit message: Updated: Kicad libraries for Schematic and PCB
Parts:
- removed Q5: NMOS, SSM3K324R,LF:SOT-23F_TOS-M
- added Q1: SSM3K341R_LF, SSM3K341R:SOT-23F_TOS, F.Cu at (43.4, 64.2)
- D3, D5, D7, D9: value IR R -> D_Photo
- Q2, Q3, Q4: value NMOS -> SSM3K341R_LF; footprint SSM3K324R,LF:SOT-23F_TOS-M -> SSM3K341R:SOT-23F_TOS
- moved Q4 27.3 mm to (117.5, 70.7)
- moved Q2 27.2 mm to (70.0, 57.7)
- moved Q3 23.0 mm to (93.3, 57.9), turned to 0 degrees
- moved C10 2.33 mm to (87.1, 86.9)
- moved C9 1.96 mm to (84.9, 86.9)
Connections:
- Q2 pad 1: Net-(D2-K) -> Net-(Q2-Pad1)
- Q2 pad 2: Net-(Q2-G) -> GND
- Q2 pad 3: GND -> Net-(D4-K)
- Q3 pad 1: Net-(D4-K) -> Net-(Q3-Pad1)
- Q3 pad 2: Net-(Q3-G) -> GND
- Q3 pad 3: GND -> Net-(D6-K)
- Q4 pad 1: Net-(D6-K) -> Net-(Q4-Pad1)
- Q4 pad 2: Net-(Q4-G) -> GND
- Q4 pad 3: GND -> Net-(D8-K)
- R18 pad 1: Net-(Q2-G) -> Net-(Q1-Pad1)
- R20 pad 1: Net-(Q2-G) -> Net-(Q1-Pad1)
- R22 pad 1: Net-(Q3-G) -> Net-(Q2-Pad1)
- R23 pad 1: Net-(Q3-G) -> Net-(Q2-Pad1)
- R26 pad 1: Net-(Q4-G) -> Net-(Q3-Pad1)
- R27 pad 1: Net-(Q4-G) -> Net-(Q3-Pad1)
- R30 pad 1: Net-(Q5-G) -> Net-(Q4-Pad1)
- R31 pad 1: Net-(Q5-G) -> Net-(Q4-Pad1)
Routing:
- net Net-(Q4-Pad1): track 0.00 -> 8.00 mm
- net Net-(Q2-G): track 7.95 -> 0.00 mm
- net Net-(Q1-Pad1): track 0.00 -> 7.94 mm
- net Net-(Q5-G): track 7.83 -> 0.00 mm
- net Net-(Q3-G): track 5.61 -> 0.00 mm
- net Net-(Q2-Pad1): track 0.00 -> 5.61 mm
- net Net-(Q3-Pad1): track 0.00 -> 5.56 mm
- net Net-(Q4-G): track 5.54 -> 0.00 mm
- net REGOUT2: track 9.22 -> 6.89 mm
- net REGOUT1: track 8.76 -> 6.97 mm
- net GND: track 63.6 -> 63.4 mm, vias 76 -> 84
