File: hardware/pcb/TMPM4KNF10AFG.kicad_sch (KiCad schematic)
At the start: 91 parts, among them J1 Conn_01x02_Socket, J2 Conn_01x02_Socket, J3 Conn_01x02_Socket, J4 Conn_01x06_Pin, J5 Conn_01x03_Pin, J6 Conn_01x06_Pin, J7 Conn_01x06_Pin, J8 Conn_01x04_Pin, Q2 NMOS, Q3 NMOS, Q4 NMOS, Q5 NMOS, SW1 CSS-1210MC, SW2 EVQ-PBG05R, U1 TMPM4KNF10AFG, U2 BD9C301FJ-E2, U4 TB67H450AFNG_EL, U5 TB67H450AFNG_EL

Commit message: Updated: Kicad libraries for Schematic and PCB
Parts:
- removed D3, D5, D7, D9: IR R, LED_THT:LED_D5.0mm_Horizontal_O1.27mm_Z3.0mm_IRBlack, symbol Device:D
- removed Q2, Q3, Q4, Q5: NMOS, SSM3K324R,LF:SOT-23F_TOS-M, symbol Simulation_SPICE:NMOS
- added D3, D5, D7, D9: D_Photo, LED_THT:LED_D5.0mm_Horizontal_O1.27mm_Z3.0mm_IRBlack, symbol Device:D_Photo
- added Q1, Q2, Q3, Q4: SSM3K341R_LF, SSM3K341R:SOT-23F_TOS, symbol SSM3K341R:SSM3K341R_LF
Connections:
- net GND: now also D3.2 (A), D5.2 (A), D7.2 (A), D9.2 (A), Q1.2, Q2.2, Q3.2, Q4.2
- net IR_OUT0: now also D3.1 (K)
- net IR_OUT1: now also D5.1 (K)
- net IR_OUT2: now also D7.1 (K)
- net IR_OUT3: now also D9.1 (K)
- net at D4.1 (K): now also Q2.3
- net at R30.1, R31.1: now also Q4.1
- net at D2.1 (K): now also Q1.3
- net at D6.1 (K): now also Q3.3
- net at R26.1, R27.1: now also Q3.1
- net at D8.1 (K): now also Q4.3
- net at R22.1, R23.1: now also Q2.1
- net at R18.1, R20.1: now also Q1.1
Other:
- moved on the sheet: R18, R20, R22, R23, R26, R27, R30, R31
